File: PCB/zetaboard/zetaboard.kicad_pcb (KiCad board)
At the start: 2 copper layers, 116 parts, among them SW1 RotaryEncoder_Switch, SW2 RotaryEncoder_Switch, U1 Raspberry_Pi_Pico_2W

Commit message: Schematic finished and PCB started.
Parts:
- added C1: C, Capacitor_SMD:C_0805_2012Metric, F.Cu at (134.9, 124.1)
- added C10: C, Capacitor_SMD:C_0805_2012Metric, F.Cu at (12.1, 170.0)
- added C11: C, Capacitor_SMD:C_0805_2012Metric, F.Cu at (16.5, 142.9)
- added C12: C, Capacitor_SMD:C_0805_2012Metric, F.Cu at (16.5, 145.9)
- added C13: C, Capacitor_SMD:C_0805_2012Metric, F.Cu at (16.5, 148.9)
- added C14: C, Capacitor_SMD:C_0805_2012Metric, F.Cu at (16.5, 152.0)
- added C15: C, Capacitor_SMD:C_0805_2012Metric, F.Cu at (16.5, 155.0)
- added C16: C, Capacitor_SMD:C_0805_2012Metric, F.Cu at (16.5, 158.0)
- added C17: C, Capacitor_SMD:C_0805_2012Metric, F.Cu at (16.5, 161.0)
- added C18: C, Capacitor_SMD:C_0805_2012Metric, F.Cu at (16.5, 164.0)
- added C19: C, Capacitor_SMD:C_0805_2012Metric, F.Cu at (16.5, 167.0)
- added C2: C, Capacitor_SMD:C_0805_2012Metric, F.Cu at (154.0, 124.1)
- added C20: C, Capacitor_SMD:C_0805_2012Metric, F.Cu at (16.5, 170.0)
- added C21: C, Capacitor_SMD:C_0805_2012Metric, F.Cu at (21.0, 142.9)
- added C22: C, Capacitor_SMD:C_0805_2012Metric, F.Cu at (21.0, 145.9)
- added C23: C, Capacitor_SMD:C_0805_2012Metric, F.Cu at (21.0, 148.9)
- added C24: C, Capacitor_SMD:C_0805_2012Metric, F.Cu at (21.0, 152.0)
- added C25: C, Capacitor_SMD:C_0805_2012Metric, F.Cu at (21.0, 155.0)
- added C26: C, Capacitor_SMD:C_0805_2012Metric, F.Cu at (21.0, 158.0)
- added C27: C, Capacitor_SMD:C_0805_2012Metric, F.Cu at (21.0, 161.0)
- added C28: C, Capacitor_SMD:C_0805_2012Metric, F.Cu at (21.0, 164.0)
- added C29: C, Capacitor_SMD:C_0805_2012Metric, F.Cu at (21.0, 167.0)
- added C3: C, Capacitor_SMD:C_0805_2012Metric, F.Cu at (12.1, 148.9)
- added C30: C, Capacitor_SMD:C_0805_2012Metric, F.Cu at (21.0, 170.0)
- added C31: C, Capacitor_SMD:C_0805_2012Metric, F.Cu at (25.4, 142.9)
- added C32: C, Capacitor_SMD:C_0805_2012Metric, F.Cu at (25.4, 145.9)
- added C33: C, Capacitor_SMD:C_0805_2012Metric, F.Cu at (25.4, 148.9)
- added C34: C, Capacitor_SMD:C_0805_2012Metric, F.Cu at (25.4, 152.0)
- added C35: C, Capacitor_SMD:C_0805_2012Metric, F.Cu at (25.4, 155.0)
- added C36: C, Capacitor_SMD:C_0805_2012Metric, F.Cu at (25.4, 158.0)
- added C37: C, Capacitor_SMD:C_0805_2012Metric, F.Cu at (25.4, 161.0)
- added C38: C, Capacitor_SMD:C_0805_2012Metric, F.Cu at (25.4, 164.0)
- added C39: C, Capacitor_SMD:C_0805_2012Metric, F.Cu at (25.4, 167.0)
- added C4: C, Capacitor_SMD:C_0805_2012Metric, F.Cu at (12.1, 152.0)
- added C40: C, Capacitor_SMD:C_0805_2012Metric, F.Cu at (25.4, 170.0)
- added C41: C, Capacitor_SMD:C_0805_2012Metric, F.Cu at (29.9, 142.9)
- added C42: C, Capacitor_SMD:C_0805_2012Metric, F.Cu at (29.9, 145.9)
- added C43: C, Capacitor_SMD:C_0805_2012Metric, F.Cu at (29.9, 148.9)
- added C44: C, Capacitor_SMD:C_0805_2012Metric, F.Cu at (29.9, 152.0)
- added C45: C, Capacitor_SMD:C_0805_2012Metric, F.Cu at (29.9, 155.0)
- added C46: C, Capacitor_SMD:C_0805_2012Metric, F.Cu at (29.9, 158.0)
- added C47: C, Capacitor_SMD:C_0805_2012Metric, F.Cu at (29.9, 161.0)
- added C48: C, Capacitor_SMD:C_0805_2012Metric, F.Cu at (29.9, 164.0)
- added C49: C, Capacitor_SMD:C_0805_2012Metric, F.Cu at (29.9, 167.0)
- added C5: C, Capacitor_SMD:C_0805_2012Metric, F.Cu at (12.1, 155.0)
- added C50: C, Capacitor_SMD:C_0805_2012Metric, F.Cu at (29.9, 170.0)
- added C51: C, Capacitor_SMD:C_0805_2012Metric, F.Cu at (34.3, 142.9)
- added C52: C, Capacitor_SMD:C_0805_2012Metric, F.Cu at (34.3, 145.9)
- added C53: C, Capacitor_SMD:C_0805_2012Metric, F.Cu at (34.3, 148.9)
- added C54: C, Capacitor_SMD:C_0805_2012Metric, F.Cu at (34.3, 152.0)
- added C55: C, Capacitor_SMD:C_0805_2012Metric, F.Cu at (34.3, 155.0)
- added C56: C, Capacitor_SMD:C_0805_2012Metric, F.Cu at (34.3, 158.0)
- added C57: C, Capacitor_SMD:C_0805_2012Metric, F.Cu at (34.3, 161.0)
- added C58: C, Capacitor_SMD:C_0805_2012Metric, F.Cu at (34.3, 164.0)
- added C59: C, Capacitor_SMD:C_0805_2012Metric, F.Cu at (34.3, 167.0)
- added C6: C, Capacitor_SMD:C_0805_2012Metric, F.Cu at (12.1, 158.0)
- added C7: C, Capacitor_SMD:C_0805_2012Metric, F.Cu at (12.1, 161.0)
- added C8: C, Capacitor_SMD:C_0805_2012Metric, F.Cu at (12.1, 164.0)
- added C9: C, Capacitor_SMD:C_0805_2012Metric, F.Cu at (12.1, 167.0)
- added D113: SK6812MINI, LED_SMD:LED_SK6812MINI_PLCC4_3.5x3.5mm_P1.75mm, F.Cu at (424.7, 131.5)
- added D114: SK6812MINI, LED_SMD:LED_SK6812MINI_PLCC4_3.5x3.5mm_P1.75mm, F.Cu at (424.7, 141.1)
- added R1: Resistor, Resistor_SMD:R_0805_2012Metric, F.Cu at (130.2, 124.1)
- added S1: Keyswitch, ScottoKeebs_Hotswap:Hotswap_MX_1.00u, F.Cu at (140.7, 114.6)
- added S10: Keyswitch, ScottoKeebs_Hotswap:Hotswap_MX_1.00u, F.Cu at (312.1, 114.6)
- added S11: Keyswitch, ScottoKeebs_Hotswap:Hotswap_MX_2.00u, F.Cu at (340.7, 114.6)
- added S12: Keyswitch, ScottoKeebs_Hotswap:Hotswap_MX_1.50u, F.Cu at (107.3, 133.7)
- added S13: Keyswitch, ScottoKeebs_Hotswap:Hotswap_MX_1.00u, F.Cu at (131.1, 133.7)
- added S14: Keyswitch, ScottoKeebs_Hotswap:Hotswap_MX_1.00u, F.Cu at (150.2, 133.7)
- added S15: Keyswitch, ScottoKeebs_Hotswap:Hotswap_MX_1.00u, F.Cu at (169.2, 133.7)
- added S16: Keyswitch, ScottoKeebs_Hotswap:Hotswap_MX_1.00u, F.Cu at (188.3, 133.7)
- added S17: Keyswitch, ScottoKeebs_Hotswap:Hotswap_MX_1.00u, F.Cu at (207.3, 133.7)
- added S18: Keyswitch, ScottoKeebs_Hotswap:Hotswap_MX_1.00u, F.Cu at (226.4, 133.7)
- added S19: Keyswitch, ScottoKeebs_Hotswap:Hotswap_MX_1.00u, F.Cu at (245.4, 133.7)
- added S2: Keyswitch, ScottoKeebs_Hotswap:Hotswap_MX_1.00u, F.Cu at (159.7, 114.6)
- added S20: Keyswitch, ScottoKeebs_Hotswap:Hotswap_MX_1.00u, F.Cu at (264.5, 133.7)
- added S21: Keyswitch, ScottoKeebs_Hotswap:Hotswap_MX_1.00u, F.Cu at (283.5, 133.7)
- added S22: Keyswitch, ScottoKeebs_Hotswap:Hotswap_MX_1.00u, F.Cu at (302.6, 133.7)
- added S23: Keyswitch, ScottoKeebs_Hotswap:Hotswap_MX_1.25u, F.Cu at (324.0, 133.7)
- added S24: Keyswitch, ScottoKeebs_Hotswap:Hotswap_MX_1.25u, F.Cu at (347.8, 133.7)
- added S26: Keyswitch, ScottoKeebs_Hotswap:Hotswap_MX_1.00u, F.Cu at (135.9, 152.7)
- added S27: Keyswitch, ScottoKeebs_Hotswap:Hotswap_MX_1.00u, F.Cu at (154.9, 152.7)
- added S28: Keyswitch, ScottoKeebs_Hotswap:Hotswap_MX_1.00u, F.Cu at (174.0, 152.7)
- added S29: Keyswitch, ScottoKeebs_Hotswap:Hotswap_MX_1.00u, F.Cu at (193.0, 152.7)
- added S3: Keyswitch, ScottoKeebs_Hotswap:Hotswap_MX_1.00u, F.Cu at (178.8, 114.6)
- added S30: Keyswitch, ScottoKeebs_Hotswap:Hotswap_MX_1.00u, F.Cu at (212.1, 152.7)
- added S31: Keyswitch, ScottoKeebs_Hotswap:Hotswap_MX_1.00u, F.Cu at (231.1, 152.7)
- added S32: Keyswitch, ScottoKeebs_Hotswap:Hotswap_MX_1.00u, F.Cu at (250.2, 152.7)
- added S33: Keyswitch, ScottoKeebs_Hotswap:Hotswap_MX_1.00u, F.Cu at (269.2, 152.7)
- added S34: Keyswitch, ScottoKeebs_Hotswap:Hotswap_MX_1.00u, F.Cu at (288.3, 152.7)
- added S35: Keyswitch, ScottoKeebs_Hotswap:Hotswap_MX_1.00u, F.Cu at (307.3, 152.7)
- added S36: Keyswitch, ScottoKeebs_Hotswap:Hotswap_MX_2.25u, F.Cu at (338.3, 152.7)
- added S37: Keyswitch, ScottoKeebs_Hotswap:Hotswap_MX_2.25u, F.Cu at (114.5, 171.8)
- added S38: Keyswitch, ScottoKeebs_Hotswap:Hotswap_MX_1.00u, F.Cu at (145.4, 171.8)
- added S39: Keyswitch, ScottoKeebs_Hotswap:Hotswap_MX_1.00u, F.Cu at (164.5, 171.8)
- added S4: Keyswitch, ScottoKeebs_Hotswap:Hotswap_MX_1.00u, F.Cu at (197.8, 114.6)
- added S40: Keyswitch, ScottoKeebs_Hotswap:Hotswap_MX_1.00u, F.Cu at (183.5, 171.8)
- added S41: Keyswitch, ScottoKeebs_Hotswap:Hotswap_MX_1.00u, F.Cu at (202.6, 171.8)
- added S42: Keyswitch, ScottoKeebs_Hotswap:Hotswap_MX_1.00u, F.Cu at (221.6, 171.8)
- added S43: Keyswitch, ScottoKeebs_Hotswap:Hotswap_MX_1.00u, F.Cu at (240.7, 171.8)
- added S44: Keyswitch, ScottoKeebs_Hotswap:Hotswap_MX_1.00u, F.Cu at (259.7, 171.8)
- added S45: Keyswitch, ScottoKeebs_Hotswap:Hotswap_MX_1.00u, F.Cu at (278.8, 171.8)
- added S46: Keyswitch, ScottoKeebs_Hotswap:Hotswap_MX_1.00u, F.Cu at (297.8, 171.8)
- added S47: Keyswitch, ScottoKeebs_Hotswap:Hotswap_MX_1.00u, F.Cu at (316.9, 171.8)
- added S48: Keyswitch, ScottoKeebs_Hotswap:Hotswap_MX_1.00u, F.Cu at (335.9, 171.8)
- added S49: Keyswitch, ScottoKeebs_Hotswap:Hotswap_MX_1.00u, F.Cu at (102.6, 190.8)
- added S5: Keyswitch, ScottoKeebs_Hotswap:Hotswap_MX_1.00u, F.Cu at (216.9, 114.6)
- added S50: Keyswitch, ScottoKeebs_Hotswap:Hotswap_MX_1.00u, F.Cu at (121.6, 190.8)
- added S51: Keyswitch, ScottoKeebs_Hotswap:Hotswap_MX_1.00u, F.Cu at (140.7, 190.8)
- added S52: Keyswitch, ScottoKeebs_Hotswap:Hotswap_MX_1.00u, F.Cu at (159.7, 190.8)
- added S53: Keyswitch, ScottoKeebs_Hotswap:Hotswap_MX_6.25u, F.Cu at (228.8, 190.8)
- added S54: Keyswitch, ScottoKeebs_Hotswap:Hotswap_MX_1.00u, F.Cu at (297.8, 190.8)
- added S55: Keyswitch, ScottoKeebs_Hotswap:Hotswap_MX_1.00u, F.Cu at (316.9, 190.8)
- added S56: Keyswitch, ScottoKeebs_Hotswap:Hotswap_MX_1.00u, F.Cu at (335.9, 190.8)
- added S6: Keyswitch, ScottoKeebs_Hotswap:Hotswap_MX_1.00u, F.Cu at (235.9, 114.6)
- added S7: Keyswitch, ScottoKeebs_Hotswap:Hotswap_MX_1.00u, F.Cu at (255.0, 114.6)
- added S8: Keyswitch, ScottoKeebs_Hotswap:Hotswap_MX_1.00u, F.Cu at (274.0, 114.6)
- added S9: Keyswitch, ScottoKeebs_Hotswap:Hotswap_MX_1.00u, F.Cu at (293.1, 114.6)
- added U2: TM1637_Module, TM137:TM1637 Display Module, F.Cu at (107.8, 111.7)
- D58: moved to B.Cu
- moved SW2 369.9 mm to (350.0, 197.3), turned to 90 degrees
- moved SW1 368.6 mm to (350.0, 178.2), turned to 90 degrees
- moved D112 356.8 mm to (424.7, 122.0)
- moved D111 356.5 mm to (424.7, 112.5)
- moved D11 344.2 mm to (359.7, 117.5), turned to 90 degrees
- moved D36 341.5 mm to (359.7, 155.6), turned to 90 degrees
- moved D24 341.0 mm to (359.7, 136.5), turned to 90 degrees
- moved D109 322.7 mm to (389.1, 118.2)
- moved D48 320.6 mm to (338.8, 162.2), turned to 180 degrees
- moved D23 319.7 mm to (335.9, 136.5), turned to 90 degrees
- moved D47 318.0 mm to (326.4, 174.6), turned to 90 degrees
- moved D56 316.3 mm to (338.8, 181.3), turned to 180 degrees
- moved D55 313.2 mm to (326.4, 193.7), turned to 90 degrees
- moved D110 312.6 mm to (379.6, 118.2)
- moved D10 308.2 mm to (321.6, 117.5), turned to 90 degrees
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Connections:
- D112 pad 1: unconnected-(D112-DOUT-Pad1) -> Net-(D112-DOUT)
Other:
- board outline added: 300 x 119.1 mm

Commit message: Save commit just in case I mess something up with removing the capacitors
Parts:
- removed C58, C59: C, Capacitor_SMD:C_0805_2012Metric
- removed D113, D114: SK6812MINI, LED_SMD:LED_SK6812MINI_PLCC4_3.5x3.5mm_P1.75mm
- D58: moved to F.Cu
- moved D67 242.0 mm to (340.6, 119.5)
- moved D80 239.9 mm to (347.8, 138.5)
- moved D66 234.0 mm to (312.1, 119.5)
- moved D92 229.4 mm to (338.3, 157.5)
- moved D104 225.9 mm to (335.8, 176.5)
- moved D79 221.2 mm to (324.1, 138.5)
- moved D103 213.4 mm to (317.1, 176.5)
- moved D91 205.9 mm to (307.3, 157.5)
- moved D78 205.6 mm to (302.6, 138.5)
- moved D102 201.6 mm to (297.8, 176.5)
- moved D90 194.3 mm to (288.8, 157.5)
- moved D77 193.3 mm to (283.6, 138.5)
- moved D101 191.3 mm to (278.8, 176.5)
- moved C41 187.7 mm to (190.3, 45.5)
- moved C11 187.7 mm to (177.0, 45.5)
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Connections:
- D112 pad 1: Net-(D112-DOUT) -> unconnected-(D112-DOUT-Pad1)
Other:
- board size 300 x 119.1 mm -> 299 x 107.1 mm

Commit message: Still on the PCB
Parts:
- removed C1, C10, C11, C12, C13, C14, C15, C16, C17, C18, C19, C2, C20, C21, C22, C23, C24, C25, C26, C27, C28, C29, C3, C30, C31, C32, C33, C34, C35, C36, C37, C38, C39, C4, C40, C41, C42, C43, C44, C45, C46, C47, C48, C49, C5, C50, C51, C52, C53, C54, C55, C56, C57, C6, C7, C8, C9: C, Capacitor_SMD:C_0805_2012Metric
- D1, D10, D11, D12, D13, D14, D15, D16, D17, D18, D19, D2, D20, D21, D22, D23, D24, D25, D26, D27, D28, D29, D3, D30, D31, D32, D33, D34, D35, D36, D37, D38, D39, D4, D40, D41, D42, D43, D44, D45, D46, D47, D48, D49, D5, D50, D51, D52, D53, D54, D55, D56, D6, D7, D8, D9: moved to B.Cu
- moved D48 6.68 mm to (332.1, 162.2), turned to 0 degrees
- moved D56 6.68 mm to (332.1, 181.3), turned to 0 degrees
- moved U1 3.75 mm to (79.7, 129.1)
- moved R1 1.08 mm to (131.1, 123.5)
Routing:
- net GND: track 0.00 -> 1911.8 mm, vias 0 -> 1
- net Col 9: track 0.00 -> 634.0 mm
- net Col 10: track 0.00 -> 619.1 mm, vias 0 -> 2
- net Col 11: track 0.00 -> 580.6 mm, vias 0 -> 9
- net Col 12: track 0.00 -> 453.6 mm, vias 0 -> 2
- net Col 8: track 0.00 -> 402.8 mm, vias 0 -> 3
- net Col 7: track 0.00 -> 373.0 mm, vias 0 -> 3
- net Col 6: track 0.00 -> 368.3 mm
- net Col 5: track 0.00 -> 343.3 mm
- net 1B: track 0.00 -> 328.2 mm, vias 0 -> 4
- net 2A: track 0.00 -> 327.4 mm, vias 0 -> 1
- net Row 4: track 0.00 -> 321.1 mm, vias 0 -> 2
- net 2B: track 0.00 -> 320.5 mm, vias 0 -> 3
- net 1A: track 0.00 -> 302.1 mm, vias 0 -> 4
- net Row 3: track 0.00 -> 302.0 mm, vias 0 -> 2
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Other:
- board size 299 x 107.1 mm -> 295 x 100 mm
